File: design/design.kicad_sch (KiCad schematic)
At the start: 30 parts, among them J1 Conn_01x03_Pin, J2 Conn_01x02_Pin, J3 Conn_01x02_Pin, U1 MC7912, U2 L7812, U3 OPA209AID, U4 TL081, U5 TL081

Commit message: Version final, archivos Gerber exportados y enviados
Parts:
- added J4, J5: Conn_01x02_Pin, Connector_PinHeader_2.54mm:PinHeader_1x02_P2.54mm_Vertical, symbol Connector:Conn_01x02_Pin
Connections:
- net -12V: now also J5.2 (Pin_2)
- net Earth: now also J4.2 (Pin_2), J5.1 (Pin_1)
- net at R10.2, R8.1, U3.6 (OUT): now also J4.1 (Pin_1)
Changed lines of the file:
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@@
   (junction (at 121.92 95.25) (diameter 0) (color 0 0 0 0)
   )
+  (junction (at 158.75 133.35) (diameter 0) (color 0 0 0 0)
+  )
   (junction (at 85.09 116.84) (diameter 0) (color 0 0 0 0)
   )
   (junction (at 184.15 119.38) (diameter 0) (color 0 0 0 0)
   )
+  (junction (at 125.73 38.1) (diameter 0) (color 0 0 0 0)
+  )
   (junction (at 115.57 55.88) (diameter 0) (color 0 0 0 0)
   )
+  (junction (at 110.49 46.99) (diameter 0) (color 0 0 0 0)
+  )
   (junction (at 82.55 116.84) (diameter 0) (color 0 0 0 0)
   )
@@
     (stroke (width 0) (type default))
   )
+  (wire (pts (xy 158.75 133.35) (xy 158.75 135.89))
+    (stroke (width 0) (type default))
+  )
   (wire (pts (xy 82.55 111.76) (xy 82.55 116.84))
     (stroke (width 0) (type default))
@@
     (stroke (width 0) (type default))
   )
+  (wire (pts (xy 125.73 38.1) (xy 130.81 38.1))
+    (stroke (width 0) (type default))
+  )
   (wire (pts (xy 115.57 55.88) (xy 130.81 55.88))
     (stroke (width 0) (type default))
@@
     (stroke (width 0) (type default))
   )
+  (wire (pts (xy 125.73 44.45) (xy 125.73 38.1))
+    (stroke (width 0) (type default))
+  )
   (wire (pts (xy 210.82 121.92) (xy 210.82 105.41))
     (stroke (width 0) (type default))
@@
     (stroke (width 0) (type default))
   )
+  (wire (pts (xy 153.67 119.38) (xy 153.67 130.81))
+    (stroke (width 0) (type default))
+  )
   (wire (pts (xy 101.6 63.5) (xy 101.6 67.31))
     (stroke (width 0) (type default))
@@
     (stroke (width 0) (type default))
   )
+  (wire (pts (xy 153.67 133.35) (xy 158.75 133.35))
+    (stroke (width 0) (type default))
+  )
   (wire (pts (xy 184.15 105.41) (xy 184.15 119.38))
     (stroke (width 0) (type default))
@@
     (stroke (width 0) (type default))
   )
-  (wire (pts (xy 158.75 130.81) (xy 158.75 135.89))
+  (wire (pts (xy 158.75 130.81) (xy 158.75 133.35))
     (stroke (width 0) (type default))
   )
@@
     (stroke (width 0) (type default))
   )
-  (wire (pts (xy 115.57 38.1) (xy 130.81 38.1))
+  (wire (pts (xy 115.57 38.1) (xy 125.73 38.1))
+    (stroke (width 0) (type default))
+  )
+  (wire (pts (xy 110.49 46.99) (xy 125.73 46.99))
     (stroke (width 0) (type default))
   )
@@
     )
   )
+  (symbol (lib_id "Connector:Conn_01x02_Pin") (at 148.59 130.81 0) (unit 1)
+    (in_bom yes) (on_board yes) (dnp no) (fields_autoplaced)
+    (property "Reference" "J4" (at 149.225 125.73 0)
+      (effects (font (size 1.27 1.27)))
+    )
+    (property "Value" "Conn_01x02_Pin" (at 149.225 128.27 0)
+      (effects (font (size 1.27 1.27)))
+    )
+    (property "Footprint" "Connector_PinHeader_2.54mm:PinHeader_1x02_P2.54mm_Vertical" (at 148.59 130.81 0)
+      (effects (font (size 1.27 1.27)) hide)
+    )
+    (property "Datasheet" "~" (at 148.59 130.81 0)
+      (effects (font (size 1.27 1.27)) hide)
+    )
+    (pin "1")
+    (pin "2")
+    (instances
+      (project "design"
+        (path "/a520f27b-3eb4-44e7-9faf-250bc52b55ee"
+          (reference "J4") (unit 1)
+        )
+      )
+    )
+  )
   (symbol (lib_id "Device:R_US") (at 176.53 119.38 270) (unit 1)
     (in_bom yes) (on_board yes) (dnp no) (fields_autoplaced)
@@
         )
       )
+    )
+  )
+  (symbol (lib_id "Connector:Conn_01x02_Pin") (at 130.81 46.99 180) (unit 1)
+    (in_bom yes) (on_board yes) (dnp no)
+    (property "Reference" "J5" (at 132.08 44.45 0)
+      (effects (font (size 1.27 1.27)) (justify right))
+    )
+    (property "Value" "Conn_01x02_Pin" (at 121.92 48.26 0)
+      (effects (font (size 1.27 1.27)) (justify right))
+    )
+    (property "Footprint" "Connector_PinHeader_2.54mm:PinHeader_1x02_P2.54mm_Vertical" (at 130.81 46.99 0)
+      (effects (font (size 1.27 1.27)) hide)
+    )
+    (property "Datasheet" "~" (at 130.81 46.99 0)
+      (effects (font (size 1.27 1.27)) hide)
+    )
+    (pin "1")
+    (pin "2")
+    (instances
+      (project "design"
+        (path "/a520f27b-3eb4-44e7-9faf-250bc52b55ee"
+          (reference "J5") (unit 1)
+        )
+      )
